File: DynOSSAT-EDU-EPS.kicad_pcb (KiCad board)
At the start: 4 copper layers, 42 x 42 mm, 111 parts, among them J1 Conn_01x05_Female, J2 USB_C_Receptacle_USB2.0, J4 PV Panel 1, J5 PV Panel 2, J6 Battery, J7 Conn_02x20_Odd_Even, J8 Conn_02x20_Odd_Even, Q1 SQ3989EV, Q2 DMG2305, SW1 SW_Push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

Commit message: Change MISO/MOSI for SDI/SDO
Update library to latest version
Parts:
- J4, J5, J6: footprint Connector_Molex:Molex_PicoBlade_53048-0210_1x02_P1.25mm_Horizontal -> DynOSSAT:Molex_PicoBlade_53048-0210_1x02_P1.25mm_Horizontal
- U8: footprint Package_DFN_QFN:VQFN-16-1EP_3x3mm_P0.5mm_EP1.45x1.45mm -> DynOSSAT:VQFN-16-1EP_3x3mm_P0.5mm_EP1.45x1.45mm
